File: MotorDriver1/untitled.kicad_sch (KiCad schematic)
At the start: 9 parts, among them U2 MCP2562FDT-H/SN, U3 MCP2562FDT-H/SN, U4 XIAO-ESP32-C5-DIP

Commit message: Updated footprints
Parts:
- renumbered C12 to C15, C13 to C16, R14 to R16, R15 to R17, R17 to R18, R16 to R19, U4 to U2, U2 to U3, U3 to U4
Changed lines of the file:
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@@
 		(dnp no)
 		(fields_autoplaced yes)
-		(property "Reference" "R16"
+		(property "Reference" "R19"
 			(at 171.45 52.0699 0)
 			(effects
@@
 			(project "MotorDriver1"
 				(path "/79cc9cfe-04d6-4d00-aa84-feae66cf8c45/72c1ec77-4632-4600-a6d8-99c07ceb64a9"
-					(reference "R16")
+					(reference "R19")
 					(unit 1)
 				)
@@
 		(dnp no)
 		(fields_autoplaced yes)
-		(property "Reference" "#PWR040"
+		(property "Reference" "#PWR045"
 			(at 33.02 60.96 0)
 			(effects
@@
 			(project "MotorDriver1"
 				(path "/79cc9cfe-04d6-4d00-aa84-feae66cf8c45/72c1ec77-4632-4600-a6d8-99c07ceb64a9"
-					(reference "#PWR040")
+					(reference "#PWR045")
 					(unit 1)
 				)
@@
 		(dnp no)
 		(fields_autoplaced yes)
-		(property "Reference" "#PWR041"
+		(property "Reference" "#PWR046"
 			(at 64.77 63.5 0)
 			(effects
@@
 			(project "MotorDriver1"
 				(path "/79cc9cfe-04d6-4d00-aa84-feae66cf8c45/72c1ec77-4632-4600-a6d8-99c07ceb64a9"
-					(reference "#PWR041")
+					(reference "#PWR046")
 					(unit 1)
 				)
@@
 		(dnp no)
 		(fields_autoplaced yes)
-		(property "Reference" "#PWR043"
+		(property "Reference" "#PWR050"
 			(at 173.99 63.5 0)
 			(effects
@@
 			(project "MotorDriver1"
 				(path "/79cc9cfe-04d6-4d00-aa84-feae66cf8c45/72c1ec77-4632-4600-a6d8-99c07ceb64a9"
-					(reference "#PWR043")
+					(reference "#PWR050")
 					(unit 1)
 				)
@@
 		(dnp no)
 		(fields_autoplaced yes)
-		(property "Reference" "C13"
+		(property "Reference" "C16"
 			(at 200.66 49.5299 0)
 			(effects
@@
 			(project "MotorDriver1"
 				(path "/79cc9cfe-04d6-4d00-aa84-feae66cf8c45/72c1ec77-4632-4600-a6d8-99c07ceb64a9"
-					(reference "C13")
+					(reference "C16")
 					(unit 1)
 				)
@@
 		(dnp no)
 		(fields_autoplaced yes)
-		(property "Reference" "#PWR044"
+		(property "Reference" "#PWR049"
 			(at 154.94 60.96 0)
 			(effects
@@
 			(project "MotorDriver1"
 				(path "/79cc9cfe-04d6-4d00-aa84-feae66cf8c45/72c1ec77-4632-4600-a6d8-99c07ceb64a9"
-					(reference "#PWR044")
+					(reference "#PWR049")
 					(unit 1)
 				)
@@
 		(dnp no)
 		(fields_autoplaced yes)
-		(property "Reference" "R15"
+		(property "Reference" "R17"
 			(at 107.95 44.4499 0)
 			(effects
@@
 			(project "MotorDriver1"
 				(path "/79cc9cfe-04d6-4d00-aa84-feae66cf8c45/72c1ec77-4632-4600-a6d8-99c07ceb64a9"
-					(reference "R15")
+					(reference "R17")
 					(unit 1)
 				)
@@
 		(dnp no)
 		(fields_autoplaced yes)
-		(property "Reference" "R17"
+		(property "Reference" "R18"
 			(at 130.81 44.4499 0)
 			(effects
@@
 			(project "MotorDriver1"
 				(path "/79cc9cfe-04d6-4d00-aa84-feae66cf8c45/72c1ec77-4632-4600-a6d8-99c07ceb64a9"
-					(reference "R17")
+					(reference "R18")
 					(unit 1)
 				)
@@
 		(dnp no)
 		(fields_autoplaced yes)
-		(property "Reference" "U4"
+		(property "Reference" "U2"
 			(at 72.39 93.98 0)
 			(effects
@@
 			(project ""
 				(path "/79cc9cfe-04d6-4d00-aa84-feae66cf8c45/72c1ec77-4632-4600-a6d8-99c07ceb64a9"
-					(reference "U4")
+					(reference "U2")
 					(unit 1)
 				)
@@
 		(dnp no)
 		(fields_autoplaced yes)
-		(property "Reference" "U2"
+		(property "Reference" "U3"
 			(at 85.9633 31.75 0)
 			(effects
@@
 			(project ""
 				(path "/79cc9cfe-04d6-4d00-aa84-feae66cf8c45/72c1ec77-4632-4600-a6d8-99c07ceb64a9"
-					(reference "U2")
+					(reference "U3")
 					(unit 1)
 				)
@@
 		(dnp no)
 		(fields_autoplaced yes)
-		(property "Reference" "U3"
+		(property "Reference" "U4"
 			(at 152.7967 31.75 0)
 			(effects
@@
 			(project "MotorDriver1"
 				(path "/79cc9cfe-04d6-4d00-aa84-feae66cf8c45/72c1ec77-4632-4600-a6d8-99c07ceb64a9"
-					(reference "U3")
+					(reference "U4")
 					(unit 1)
 				)
@@
 		(dnp no)
 		(fields_autoplaced yes)
-		(property "Reference" "C12"
+		(property "Reference" "C15"
 			(at 36.83 49.5299 0)
 			(effects
@@
 			(project ""
 				(path "/79cc9cfe-04d6-4d00-aa84-feae66cf8c45/72c1ec77-4632-4600-a6d8-99c07ceb64a9"
-					(reference "C12")
+					(reference "C15")
 					(unit 1)
 				)
@@
 		(dnp no)
 		(fields_autoplaced yes)
-		(property "Reference" "#PWR039"
+		(property "Reference" "#PWR047"
 			(at 83.82 60.96 0)
 			(effects
@@
 			(project ""
 				(path "/79cc9cfe-04d6-4d00-aa84-feae66cf8c45/72c1ec77-4632-4600-a6d8-99c07ceb64a9"
-					(reference "#PWR039")
+					(reference "#PWR047")
 					(unit 1)
 				)
@@
 		(dnp no)
 		(fields_autoplaced yes)
-		(property "Reference" "#PWR045"
+		(property "Reference" "#PWR048"
 			(at 97.79 105.41 0)
 			(effects
@@
 			(project "MotorDriver1"
 				(path "/79cc9cfe-04d6-4d00-aa84-feae66cf8c45/72c1ec77-4632-4600-a6d8-99c07ceb64a9"
-					(reference "#PWR045")
+					(reference "#PWR048")
 					(unit 1)
 				)
@@
 		(dnp no)
 		(fields_autoplaced yes)
-		(property "Reference" "R14"
+		(property "Reference" "R16"
 			(at 67.31 52.0699 0)
 			(effects
@@
 			(project ""
 				(path "/79cc9cfe-04d6-4d00-aa84-feae66cf8c45/72c1ec77-4632-4600-a6d8-99c07ceb64a9"
-					(reference "R14")
+					(reference "R16")
 					(unit 1)
 				)
@@
 		(dnp no)
 		(fields_autoplaced yes)
-		(property "Reference" "#PWR042"
+		(property "Reference" "#PWR051"
 			(at 204.47 60.96 0)
 			(effects
@@
 			(project "MotorDriver1"
 				(path "/79cc9cfe-04d6-4d00-aa84-feae66cf8c45/72c1ec77-4632-4600-a6d8-99c07ceb64a9"
-					(reference "#PWR042")
-					(unit 1)
-				)
+					(reference "#PWR051")
+					(unit 1)
+				)

Commit message: assigned eo footprints
Parts:
- C15: footprint (none) -> Capacitor_SMD:C_0201_0603Metric
- C16: footprint (none) -> Capacitor_SMD:C_0402_1005Metric
- R16, R17, R18, R19: footprint (none) -> Resistor_SMD:R_0402_1005Metric
Changed lines of the file:
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@@
 			)
 		)
-		(property "Footprint" ""
+		(property "Footprint" "Resistor_SMD:R_0402_1005Metric"
 			(at 175.768 53.34 90)
 			(effects
@@
 			)
 		)
-		(property "Footprint" ""
+		(property "Footprint" "Capacitor_SMD:C_0402_1005Metric"
 			(at 203.5048 54.61 0)
 			(effects
@@
 			)
 		)
-		(property "Footprint" ""
+		(property "Footprint" "Resistor_SMD:R_0402_1005Metric"
 			(at 103.632 45.72 90)
 			(effects
@@
 			)
 		)
-		(property "Footprint" ""
+		(property "Footprint" "Resistor_SMD:R_0402_1005Metric"
 			(at 135.128 45.72 90)
 			(effects
@@
 			)
 		)
-		(property "Footprint" ""
+		(property "Footprint" "Capacitor_SMD:C_0201_0603Metric"
 			(at 33.9852 54.61 0)
 			(effects
@@
 			)
 		)
-		(property "Footprint" ""
+		(property "Footprint" "Resistor_SMD:R_0402_1005Metric"
 			(at 62.992 53.34 90)
 			(effects

Commit message: laid out PCB
Parts:
- renumbered R16 to R20, R17 to R21, R18 to R22, R19 to R23, U2 to U3, U3 to U4, U4 to U5
Changed lines of the file:
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@@
 		(dnp no)
 		(fields_autoplaced yes)
-		(property "Reference" "R19"
+		(property "Reference" "R23"
 			(at 171.45 52.0699 0)
 			(effects
@@
 			(project "MotorDriver1"
 				(path "/79cc9cfe-04d6-4d00-aa84-feae66cf8c45/72c1ec77-4632-4600-a6d8-99c07ceb64a9"
-					(reference "R19")
+					(reference "R23")
 					(unit 1)
 				)
@@
 		(dnp no)
 		(fields_autoplaced yes)
-		(property "Reference" "R17"
+		(property "Reference" "R21"
 			(at 107.95 44.4499 0)
 			(effects
@@
 			(project "MotorDriver1"
 				(path "/79cc9cfe-04d6-4d00-aa84-feae66cf8c45/72c1ec77-4632-4600-a6d8-99c07ceb64a9"
-					(reference "R17")
+					(reference "R21")
 					(unit 1)
 				)
@@
 		(dnp no)
 		(fields_autoplaced yes)
-		(property "Reference" "R18"
+		(property "Reference" "R22"
 			(at 130.81 44.4499 0)
 			(effects
@@
 			(project "MotorDriver1"
 				(path "/79cc9cfe-04d6-4d00-aa84-feae66cf8c45/72c1ec77-4632-4600-a6d8-99c07ceb64a9"
-					(reference "R18")
+					(reference "R22")
 					(unit 1)
 				)
@@
 		(dnp no)
 		(fields_autoplaced yes)
-		(property "Reference" "U2"
+		(property "Reference" "U3"
 			(at 72.39 93.98 0)
 			(effects
@@
 			(project ""
 				(path "/79cc9cfe-04d6-4d00-aa84-feae66cf8c45/72c1ec77-4632-4600-a6d8-99c07ceb64a9"
-					(reference "U2")
+					(reference "U3")
 					(unit 1)
 				)
@@
 		(dnp no)
 		(fields_autoplaced yes)
-		(property "Reference" "U3"
+		(property "Reference" "U4"
 			(at 85.9633 31.75 0)
 			(effects
@@
 			(project ""
 				(path "/79cc9cfe-04d6-4d00-aa84-feae66cf8c45/72c1ec77-4632-4600-a6d8-99c07ceb64a9"
-					(reference "U3")
+					(reference "U4")
 					(unit 1)
 				)
@@
 		(dnp no)
 		(fields_autoplaced yes)
-		(property "Reference" "U4"
+		(property "Reference" "U5"
 			(at 152.7967 31.75 0)
 			(effects
@@
 			(project "MotorDriver1"
 				(path "/79cc9cfe-04d6-4d00-aa84-feae66cf8c45/72c1ec77-4632-4600-a6d8-99c07ceb64a9"
-					(reference "U4")
+					(reference "U5")
 					(unit 1)
 				)
@@
 		(dnp no)
 		(fields_autoplaced yes)
-		(property "Reference" "R16"
+		(property "Reference" "R20"
 			(at 67.31 52.0699 0)
 			(effects
@@
 			(project ""
 				(path "/79cc9cfe-04d6-4d00-aa84-feae66cf8c45/72c1ec77-4632-4600-a6d8-99c07ceb64a9"
-					(reference "R16")
-					(unit 1)
-				)
+					(reference "R20")
+					(unit 1)
+				)

Commit message: Re-layed out eo stuff
Connections:
- net FDCAN_STM renamed FDCAN_RX_STM
Changed lines of the file:
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@@
 		)
 	)
-	(global_label "FDCAN_STM"
+	(global_label "FDCAN_RX_STM"
 		(shape output)
 		(at 71.12 41.91 180)
@@
 		)
 		(property "Intersheetrefs" "${INTERSHEET_REFS}"
-			(at 57.491 41.91 0)
+			(at 54.0439 41.91 0)
 			(effects
 				(font
@@
 		(fields_autoplaced yes)
 		(property "Reference" "U5"
-			(at 152.7967 31.75 0)
-			(effects
-				(font
-					(size 1.27 1.27)
-				)
-				(justify left)
+			(at 158.0581 31.75 0)
+			(effects
+				(font
+					(size 1.27 1.27)
+				)
+				(justify right)
 			)
 		)
 		(property "Value" "MCP2562FDT-H/SN"
-			(at 152.7967 34.29 0)
-			(effects
-				(font
-					(size 1.27 1.27)
-				)
-				(justify left)
-			)
-		)
+			(at 158.0581 34.29 0)
+			(effects
+				(font
+					(size 1.27 1.27)
+				)
+				(justify right)
+			)
+		)

Commit message: Exported final JLCPCB files
Parts:
- added C18, C19: 100 nF, Capacitor_SMD:C_0402_1005Metric, symbol Device:C
- C15: value 100nF -> 100 nF; footprint Capacitor_SMD:C_0201_0603Metric -> Capacitor_SMD:C_0402_1005Metric
- C16: value 100nF -> 100 nF
Connections:
- net 5V: now also C18.1, C19.1
- net GND: now also C18.2, C19.2
- net CANH renamed CAN_P
- net CANL renamed CAN_N
